File: totoro/totoro.sch (KiCad schematic (older format))
At the start: 81 parts, among them J1 USB_B_Micro, J2 SWR201-NRTN-S02-SA-WH, J3 SWR201-NRTN-S02-SA-WH, Q1 MMBT3904, Q2 MMBT3904, Q3 MMBT3904, Q4 2N7002, Q5 2N7002, Q6 MMBT3904, Q7 BC817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

Commit message: All parts are in the circle
Parts:
- removed C27: 100nF, Capacitor_SMD:C_0603_1608Metric, symbol Device:C
- removed Q4: 2N7002, Package_TO_SOT_SMD:SOT-23, symbol Transistor_FET:2N7002
- added C29, C30, C31, C32: 100nF, Capacitor_SMD:C_0603_1608Metric_Pad1.05x0.95mm_HandSolder, symbol Device:C
- added R30: 7.5, Resistor_SMD:R_2512_6332Metric, symbol Device:R_US
- C1: footprint Capacitor_SMD:C_0603_1608Metric -> Capacitor_SMD:C_0805_2012Metric
- R10: value 10k -> 1k; footprint Resistor_SMD:R_0603_1608Metric -> Resistor_SMD:R_0603_1608Metric_Pad1.05x0.95mm_HandSolder
- R24: value 3.71 -> 7.5; footprint Resistor_SMD:R_0603_1608Metric -> Resistor_SMD:R_2512_6332Metric; Power (none) -> 1W
- R27: value 100 -> 100k; footprint Resistor_SMD:R_0603_1608Metric -> Resistor_SMD:R_0603_1608Metric_Pad1.05x0.95mm_HandSolder
Connections:
- net +3V3: now also C29.1, C30.1, C31.1, C32.1
- net +6V: now also R30.1
- net BATTERY+: no longer Q3.1 (B), Q3.3 (C)
- net GND: now also C29.2, C30.2, C31.2, C32.2; no longer R10.2
- net OFF_SIGNAL: now also Q3.1 (B), Q3.3 (C); no longer R10.1, R27.1
- net PS_ENABLE: now also C18.1, Q5.3 (D)
- net at Q8.3 (C), R24.2: now also R30.2
- net at Q5.1 (G), R12.1: now also R27.1; no longer C18.1
- net at Q6.1 (B), R13.1, R14.1: no longer Q5.3 (D)
- net at R27.2: now also C16.1, R10.1
- net at Q3.2 (E): now also R10.2; no longer C16.1
Other:
- note added: "Bypass Caps:\nPlace close to vias in the USB Data traces"
- moved on the sheet: C11, C12, C13, C14, C16, D2, D3, Q3, Q5, Q6, R11, R12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

Commit message: Routed some traces. Shrunk board outline.
Parts:
- removed C29, C30: 100nF, Capacitor_SMD:C_0603_1608Metric_Pad1.05x0.95mm_HandSolder, symbol Device:C
Changed lines of the file:
@@
 CHARGE_ENABLE
-$Comp
-L Device:C C30
-U 1 1 5D37187A
-P 4600 5450
-F 0 "C30" H 4715 5496 50  0000 L CNN
-F 1 "100nF" H 4715 5405 50  0000 L CNN
-F 2 "Capacitor_SMD:C_0603_1608Metric_Pad1.05x0.95mm_HandSolder" H 4638 5300 50  0001 C CNN
-F 3 "~" H 4600 5450 50  0001 C CNN
-	1    4600 5450
-	1    0    0    -1
-$EndComp
 $Comp
 L Device:C C31
@@
 F 3 "~" H 5500 5450 50  0001 C CNN
 	1    5500 5450
-	1    0    0    -1
-$EndComp
-$Comp
-L Device:C C29
-U 1 1 5D38062C
-P 4150 5450
-F 0 "C29" H 4265 5496 50  0000 L CNN
-F 1 "100nF" H 4265 5405 50  0000 L CNN
-F 2 "Capacitor_SMD:C_0603_1608Metric_Pad1.05x0.95mm_HandSolder" H 4188 5300 50  0001 C CNN
-F 3 "~" H 4150 5450 50  0001 C CNN
-	1    4150 5450
-	1    0    0    -1
-$EndComp
-$Comp
-L power:GND #PWR0101
-U 1 1 5D3815BD
-P 4150 5600
-F 0 "#PWR0101" H 4150 5350 50  0001 C CNN
-F 1 "GND" H 4155 5427 50  0000 C CNN
-F 2 "" H 4150 5600 50  0001 C CNN
-F 3 "" H 4150 5600 50  0001 C CNN
-	1    4150 5600
-	1    0    0    -1
-$EndComp
-$Comp
-L power:GND #PWR0102
-U 1 1 5D3824B4
-P 4600 5600
-F 0 "#PWR0102" H 4600 5350 50  0001 C CNN
-F 1 "GND" H 4605 5427 50  0000 C CNN
-F 2 "" H 4600 5600 50  0001 C CNN
-F 3 "" H 4600 5600 50  0001 C CNN
-	1    4600 5600
 	1    0    0    -1
 $EndComp
@@
 	1    0    0    -1
 $EndComp
-$Comp
-L power:+3.3V #PWR0105
-U 1 1 5D38431F
-P 4150 5300
-F 0 "#PWR0105" H 4150 5150 50  0001 C CNN
-F 1 "+3.3V" H 4165 5473 50  0000 C CNN
-F 2 "" H 4150 5300 50  0001 C CNN
-F 3 "" H 4150 5300 50  0001 C CNN
-	1    4150 5300
-	1    0    0    -1
-$EndComp
-$Comp
-L power:+3.3V #PWR0106
-U 1 1 5D384F83
-P 4600 5300
-F 0 "#PWR0106" H 4600 5150 50  0001 C CNN
-F 1 "+3.3V" H 4615 5473 50  0000 C CNN
-F 2 "" H 4600 5300 50  0001 C CNN
-F 3 "" H 4600 5300 50  0001 C CNN
-	1    4600 5300
-	1    0    0    -1
-$EndComp

Commit message: Poured copper and stitched with vias
Parts:
- added C27, C29, C30, C33, C34, C35, C36, C37, C38, C39, C40, C41: 100nF, Capacitor_SMD:C_0603_1608Metric, symbol Device:C
Connections:
- net +3V3: now also C27.1, C29.1, C30.1, C33.1, C34.1, C35.1, C36.1, C37.1, C38.1, C39.1, C40.1, C41.1
- net GND: now also C27.2, C29.2, C30.2, C33.2, C34.2, C35.2, C36.2, C37.2, C38.2, C39.2, C40.2, C41.2
Other:
- note added: "Bonus Bypass Caps:\nPlace near signal vias or wherever\nextra bypassing may be helpful"
- moved on the sheet: C31, C32
