File: totoro/_autosave-totoro.sch (KiCad schematic (older format))
At the start: 94 parts, among them J1 USB_B_Micro, J2 SWR201-NRTN-S02-SA-WH, J3 SWR201-NRTN-S02-SA-WH, Q1 MMBT3904, Q2 MMBT3904, Q3 MMBT3904, Q5 2N7002, Q6 MMBT3904, Q7 BC817, Q8 BC817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

Commit message: Created BOM, minor value changes
Parts:
- R13: value 17.2k -> 17.4k
- R29: value 163k -> 162k
Changed lines of the file:
@@
 P 13500 3950
 F 0 "R29" V 13600 3850 50  0000 C CNN
-F 1 "163k" V 13700 3900 50  0000 C CNN
+F 1 "162k" V 13700 3900 50  0000 C CNN
 F 2 "Resistor_SMD:R_0603_1608Metric" V 13540 3940 50  0001 C CNN
 F 3 "~" H 13500 3950 50  0001 C CNN
@@
 P 8800 6650
 F 0 "R13" H 8732 6604 50  0000 R CNN
-F 1 "17.2k" H 8732 6695 50  0000 R CNN
+F 1 "17.4k" H 8732 6695 50  0000 R CNN
 F 2 "Resistor_SMD:R_0603_1608Metric" V 8840 6640 50  0001 C CNN
 F 3 "~" H 8800 6650 50  0001 C CNN
